File: 2063-Z80.kicad_pcb (KiCad board)
At the start: 4 copper layers, 100 x 100 mm, 86 parts, among them J1 Conn_01x05, J10 Conn_01x07, J11 Conn_02x03, J12 Conn_01x02, J2 DM3D-SF(41), J3 Conn_02x20, J4 Conn_02x05, J5 Conn_02x05, J6 0548190519, J7 Conn_02x13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

Commit message: Added / Changed my PCB changes.
Parts:
- added J3A1: Conn_02x02_Odd_Even, Connector_PinHeader_2.54mm:PinHeader_2x02_P2.54mm_Vertical, F.Cu at (101.9, 108.7)
- moved R2 0.66 mm to (109.5, 108.7)
- moved R6 0.66 mm to (117.6, 108.7)
- moved R1 0.66 mm to (107.4, 113.7)
- moved R3 0.66 mm to (111.5, 113.7)
- moved R4 0.66 mm to (113.5, 108.7)
- moved R5 0.66 mm to (115.6, 113.7)
Connections:
- J2 pad 1: Net-(J2-Pad1) -> (no net)
- J2 pad 8: Net-(J2-Pad8) -> (no net)
- J4 pad 1: Net-(J4-Pad1) -> (no net)
- J4 pad 10: Net-(J4-Pad10) -> (no net)
- J4 pad 2: Net-(J4-Pad2) -> (no net)
- J4 pad 4: Net-(J4-Pad4) -> (no net)
- J4 pad 6: Net-(J4-Pad6) -> (no net)
- J4 pad 7: Net-(J4-Pad7) -> (no net)
- J4 pad 8: Net-(J4-Pad8) -> (no net)
- J5 pad 1: Net-(J5-Pad1) -> (no net)
- J5 pad 10: Net-(J5-Pad10) -> (no net)
- J5 pad 2: Net-(J5-Pad2) -> (no net)
- J5 pad 4: Net-(J5-Pad4) -> (no net)
- J5 pad 6: Net-(J5-Pad6) -> (no net)
- J5 pad 7: Net-(J5-Pad7) -> (no net)
- J5 pad 8: Net-(J5-Pad8) -> (no net)
- J6 pad 2: Net-(J6-Pad2) -> (no net)
- J6 pad 3: Net-(J6-Pad3) -> (no net)
- J6 pad 4: Net-(J6-Pad4) -> (no net)
- S1 pad 1: Net-(S1-Pad1) -> (no net)
- U4 pad 7: Net-(U4-Pad7) -> (no net)
- U5 pad 10: Net-(U5-Pad10) -> (no net)
- U5 pad 11: Net-(U5-Pad11) -> (no net)
- U5 pad 17: Net-(U5-Pad17) -> (no net)
- U5 pad 24: Net-(U5-Pad24) -> (no net)
- U5 pad 29: Net-(U5-Pad29) -> (no net)
- U5 pad 30: Net-(U5-Pad30) -> (no net)
- U9 pad 10: Net-(U9-Pad10) -> /~IORQ_50
- U9 pad 9: Net-(U9-Pad9) -> /~IORQ_60
Routing:
- net /SIO_IEO: track 0.00 -> 131.1 mm, vias 0 -> 1
- net /~IORQ_60: track 0.00 -> 51.4 mm, vias 0 -> 3
- net /~IORQ_50: track 0.00 -> 51.4 mm, vias 0 -> 3
- net /SD5_MOSI: track 72.7 -> 71.2 mm
- net /SD5_CLK: track 77.4 -> 75.9 mm
- net /~SD5_SSEL: track 99.8 -> 98.4 mm
- net /~SD_SSEL: track 44.7 -> 43.8 mm
- net /A15: track 125.5 -> 126.1 mm
- net /SD_MOSI: track 51.1 -> 50.5 mm
- net GND: vias 20 -> 19
Other:
- board text added: "JLCJLCJLCJLC"
- board text added: "Rev A2063.4.3.1"
- board text added: "https://github.com/NixToDo/2063-Z80"
- board text removed: "Rev 2063.4.3.1"
- board text removed: "https://github.com/johnwinans/2063-Z80"

Commit message: Modified to fit my needs.
Routing:
- net /~IORQ_50: vias 3 -> 2
